Commit message: Update URDF: Center main robot structure and add sensor links

File: urdf/mini_bot.urdf (robot description, URDF)
Before this commit: robot mini_bot, 3 links, 2 joints
Links:
- added link camera_link
- added link imu_link
- added link range_link
Joints:
- added joint camera_joint: type fixed, parent base_link, child camera_link, origin xyz=0.105 -0.02 0.105 rpy=0 1.57 0
- added joint imu_joint: type fixed, parent base_link, child imu_link, origin xyz=0.0 0.04 0.12 rpy=0 0 0
- added joint range_joint: type fixed, parent base_link, child range_link, origin xyz=0.08 0.0 0.06 rpy=0 1.57 0
- joint left_wheel_joint: limit lower=-1000.0 upper=1000.0 effort=1.0 velocity=10.0 -> (none); origin xyz=-0.035 0.1 0.0325 rpy=0 0 0 -> xyz=0.0 0.075 0.0325 rpy=0 0 0; type revolute -> continuous
- joint right_wheel_joint: limit lower=-1000.0 upper=1000.0 effort=1.0 velocity=10.0 -> (none); origin xyz=-0.035 -0.05 0.0325 rpy=0 0 0 -> xyz=0.0 -0.075 0.0325 rpy=0 0 0; type revolute -> continuous

Commit message: Change lenght between wheels

File: urdf/mini_bot.urdf (robot description, URDF)
Before this commit: robot mini_bot, 6 links, 5 joints
Joints:
- joint left_wheel_joint: origin xyz=0.0 0.075 0.0325 rpy=0 0 0 -> xyz=0.0 0.08 0.0325 rpy=0 0 0
- joint right_wheel_joint: origin xyz=0.0 -0.075 0.0325 rpy=0 0 0 -> xyz=0.0 -0.08 0.0325 rpy=0 0 0

Commit message: Corrected range orientation

File: urdf/mini_bot.urdf (robot description, URDF)
Before this commit: robot mini_bot, 6 links, 5 joints
Joints:
- joint range_joint: origin xyz=0.08 0.0 0.06 rpy=0 1.57 0 -> xyz=0.08 0.0 0.06 rpy=0 0 0
